File: DuzaKlawiatura/Diody.kicad_sch (KiCad schematic)
At the start: 82 parts

Commit message: Added photos of layout and schematic, updated Kicad files.
Parts:
- renumbered C110 to C1010, C111 to C1011, C112 to C1012, C113 to C1013, C114 to C1014, C115 to C1015, C116 to C1016, C117 to C1017, C118 to C1018, C119 to C1019, C120 to C1020, C121 to C1021, C122 to C1022, C123 to C1023, C124 to C1024, C125 to C1025, C126 to C1026, C127 to C1027, C128 to C1028, C129 to C1029, C130 to C1030, C131 to C1031, C132 to C1032, C133 to C1033, C134 to C1034, C135 to C1035, C136 to C1036, C137 to C1037, C138 to C1038, C139 to C1039, C140 to C1040, C141 to C1041
Connections:
- net at LED16.2 (DOUT): now also LED17.4 (DIN)
- net at LED16.4 (DIN): now also LED15.2 (DOUT)
- net at LED3.2 (DOUT): now also LED4.4 (DIN)
- net at LED3.4 (DIN): now also LED2.2 (DOUT)
- net at LED24.2 (DOUT): now also LED25.4 (DIN)
- net at LED24.4 (DIN): now also LED23.2 (DOUT)
- net at LED4.2 (DOUT): now also LED5.4 (DIN)
- net at LED23.4 (DIN): now also LED22.2 (DOUT)
- net at LED5.2 (DOUT): now also LED6.4 (DIN)
- net at LED36.2 (DOUT): now also LED37.4 (DIN)
- net at LED36.4 (DIN): now also LED35.2 (DOUT)
- net at LED31.2 (DOUT): now also LED32.4 (DIN)
- net at LED31.4 (DIN): now also LED30.2 (DOUT)
- net at LED12.2 (DOUT): now also LED13.4 (DIN)
- net at LED12.4 (DIN): now also LED11.2 (DOUT)
- net at LED25.2 (DOUT): now also LED26.4 (DIN)
- net at LED33.2 (DOUT): now also LED34.4 (DIN)
- net at LED33.4 (DIN): now also LED32.2 (DOUT)
- net Sheet2: now reaches LED41.2 (DOUT)
- net at LED41.4 (DIN): now also LED40.2 (DOUT)
- net at LED40.4 (DIN): now also LED39.2 (DOUT)
- net at LED11.4 (DIN): now also LED10.2 (DOUT)
- net at LED26.2 (DOUT): now also LED27.4 (DIN)
- net at LED30.4 (DIN): now also LED29.2 (DOUT)
- net at LED2.4 (DIN): now also LED1.2 (DOUT)
- net at LED38.2 (DOUT): now also LED39.4 (DIN)
- net at LED38.4 (DIN): now also LED37.2 (DOUT)
- net at LED18.2 (DOUT): now also LED19.4 (DIN)
- net at LED18.4 (DIN): now also LED17.2 (DOUT)
- net at LED29.4 (DIN): now also LED28.2 (DOUT)
- net at LED13.2 (DOUT): now also LED14.4 (DIN)
- net at LED35.4 (DIN): now also LED34.2 (DOUT)
- net at LED28.4 (DIN): now also LED27.2 (DOUT)
- net at LED7.2 (DOUT): now also LED8.4 (DIN)
- net at LED7.4 (DIN): now also LED6.2 (DOUT)
- net at LED15.4 (DIN): now also LED14.2 (DOUT)
- net at LED8.2 (DOUT): now also LED9.4 (DIN)
- net at LED22.4 (DIN): now also LED21.2 (DOUT)
- net at LED19.2 (DOUT): now also LED20.4 (DIN)
- net at LED9.2 (DOUT): now also LED10.4 (DIN)
- net at LED21.4 (DIN): now also LED20.2 (DOUT)
