File: DuzaKlawiatura/diody1.kicad_sch (KiCad schematic)
At the start: 82 parts

Commit message: Added photos of layout and schematic, updated Kicad files.
Parts:
- renumbered C142 to C1042, C143 to C1043, C144 to C1044, C145 to C1045, C146 to C1046, C147 to C1047, C148 to C1048, C149 to C1049, C150 to C1050, C151 to C1051, C152 to C1052, C153 to C1053, C154 to C1054, C155 to C1055, C156 to C1056, C157 to C1057, C158 to C1058, C159 to C1059, C160 to C1060, C161 to C1061, C162 to C1062, C163 to C1063, C164 to C1064, C165 to C1065, C166 to C1066, C167 to C1067, C168 to C1068, C169 to C1069, C170 to C1070, C171 to C1071, C172 to C1072, C173 to C1073, C174 to C1074, C175 to C1075, C176 to C1076, C177 to C1077, C178 to C1078, C179 to C1079, C180 to C1080, C181 to C1081, C182 to C1082
Connections:
- net at LED79.2 (DOUT): now also LED80.4 (DIN)
- net at LED79.4 (DIN): now also LED78.2 (DOUT)
- net at LED53.2 (DOUT): now also LED54.4 (DIN)
- net at LED53.4 (DIN): now also LED52.2 (DOUT)
- net at LED77.2 (DOUT): now also LED78.4 (DIN)
- net at LED77.4 (DIN): now also LED76.2 (DOUT)
- net at LED70.2 (DOUT): now also LED71.4 (DIN)
- net at LED70.4 (DIN): now also LED69.2 (DOUT)
- net at LED49.2 (DOUT): now also LED50.4 (DIN)
- net at LED49.4 (DIN): now also LED48.2 (DOUT)
- net at LED42.2 (DOUT): now also LED43.4 (DIN)
- net at LED62.2 (DOUT): now also LED63.4 (DIN)
- net at LED62.4 (DIN): now also LED61.2 (DOUT)
- net at LED76.4 (DIN): now also LED75.2 (DOUT)
- net at LED55.2 (DOUT): now also LED56.4 (DIN)
- net at LED55.4 (DIN): now also LED54.2 (DOUT)
- net at LED59.2 (DOUT): now also LED60.4 (DIN)
- net at LED59.4 (DIN): now also LED58.2 (DOUT)
- net at LED65.2 (DOUT): now also LED66.4 (DIN)
- net at LED65.4 (DIN): now also LED64.2 (DOUT)
- net at LED72.2 (DOUT): now also LED73.4 (DIN)
- net at LED72.4 (DIN): now also LED71.2 (DOUT)
- net at LED51.2 (DOUT): now also LED52.4 (DIN)
- net at LED51.4 (DIN): now also LED50.2 (DOUT)
- net at LED57.2 (DOUT): now also LED58.4 (DIN)
- net at LED57.4 (DIN): now also LED56.2 (DOUT)
- net at LED63.2 (DOUT): now also LED64.4 (DIN)
- net at LED43.2 (DOUT): now also LED44.4 (DIN)
- net at LED61.4 (DIN): now also LED60.2 (DOUT)
- net at LED81.2 (DOUT): now also LED82.4 (DIN)
- net at LED81.4 (DIN): now also LED80.2 (DOUT)
- net at LED69.4 (DIN): now also LED68.2 (DOUT)
- net at LED74.2 (DOUT): now also LED75.4 (DIN)
- net at LED74.4 (DIN): now also LED73.2 (DOUT)
- net at LED68.4 (DIN): now also LED67.2 (DOUT)
- net at LED44.2 (DOUT): now also LED45.4 (DIN)
- net at LED46.2 (DOUT): now also LED47.4 (DIN)
- net at LED46.4 (DIN): now also LED45.2 (DOUT)
- net at LED47.2 (DOUT): now also LED48.4 (DIN)
- net at LED66.2 (DOUT): now also LED67.4 (DIN)
- net LED_IN renamed Sheet2
- no-connect marks 0 -> 1
