File: DuzaKlawiatura/hall.kicad_sch (KiCad schematic)
At the start: 82 parts, among them SW1 DRV5053, SW10 DRV5053, SW11 DRV5053, SW12 DRV5053, SW13 DRV5053, SW14 DRV5053, SW15 DRV5053, SW16 DRV5053, SW17 DRV5053, SW18 DRV5053, SW19 DRV5053, SW2 DRV5053, SW20 DRV5053, SW21 DRV5053, SW22 DRV5053, SW23 DRV5053, SW24 DRV5053, SW25 DRV5053, SW26 DRV5053, SW27 DRV5053, SW28 DRV5053, SW29 DRV5053, SW3 DRV5053, SW30 DRV5053, SW31 DRV5053, SW32 DRV5053, SW33 DRV5053, SW34 DRV5053, SW35 DRV5053, SW36 DRV5053, SW37 DRV5053, SW38 DRV5053, SW39 DRV5053, SW4 DRV5053, SW40 DRV5053, SW41 DRV5053, SW5 DRV5053, SW6 DRV5053, SW7 DRV5053, SW8 DRV5053, SW9 DRV5053

Commit message: Added photos of layout and schematic, updated Kicad files.
Connections:
- net SW26: now reaches SW26.2 (OUT)
- net SW37: now reaches SW37.2 (OUT)
- net SW34: now reaches SW34.2 (OUT)
- net SW30: now reaches SW30.2 (OUT)
- net SW40: now reaches SW40.2 (OUT)
- net SW2: now reaches SW2.2 (OUT)
- net SW1: now reaches SW1.2 (OUT)
- net SW29: now reaches SW29.2 (OUT)
- net SW8: now reaches SW8.2 (OUT)
- net SW5: now reaches SW5.2 (OUT)
- net SW22: now reaches SW22.2 (OUT)
- net SW3: now reaches SW3.2 (OUT)
- net SW7: now reaches SW7.2 (OUT)
- net SW11: now reaches SW11.2 (OUT)
- net SW32: now reaches SW32.2 (OUT)
- net SW33: now reaches SW33.2 (OUT)
- net SW17: now reaches SW17.2 (OUT)
- net SW21: now reaches SW21.2 (OUT)
- net SW24: now reaches SW24.2 (OUT)
- net SW38: now reaches SW38.2 (OUT)
- net SW35: now reaches SW35.2 (OUT)
- net SW9: now reaches SW9.2 (OUT)
- net SW15: now reaches SW15.2 (OUT)
- net SW36: now reaches SW36.2 (OUT)
- net SW18: now reaches SW18.2 (OUT)
- net SW19: now reaches SW19.2 (OUT)
- net SW14: now reaches SW14.2 (OUT)
- net SW27: now reaches SW27.2 (OUT)
- net SW4: now reaches SW4.2 (OUT)
- net SW39: now reaches SW39.2 (OUT)
- net SW41: now reaches SW41.2 (OUT)
- net SW13: now reaches SW13.2 (OUT)
- net SW10: now reaches SW10.2 (OUT)
- net SW23: now reaches SW23.2 (OUT)
- net SW25: now reaches SW25.2 (OUT)
- net SW12: now reaches SW12.2 (OUT)
- net SW20: now reaches SW20.2 (OUT)
- net SW6: now reaches SW6.2 (OUT)
- net SW16: now reaches SW16.2 (OUT)
- net SW31: now reaches SW31.2 (OUT)
- net SW28: now reaches SW28.2 (OUT)
