File: DuzaKlawiatura/hall1.kicad_sch (KiCad schematic)
At the start: 82 parts, among them SW42 DRV5053, SW43 DRV5053, SW44 DRV5053, SW45 DRV5053, SW46 DRV5053, SW47 DRV5053, SW48 DRV5053, SW49 DRV5053, SW50 DRV5053, SW51 DRV5053, SW52 DRV5053, SW53 DRV5053, SW54 DRV5053, SW55 DRV5053, SW56 DRV5053, SW57 DRV5053, SW58 DRV5053, SW59 DRV5053, SW60 DRV5053, SW61 DRV5053, SW62 DRV5053, SW63 DRV5053, SW64 DRV5053, SW65 DRV5053, SW66 DRV5053, SW67 DRV5053, SW68 DRV5053, SW69 DRV5053, SW70 DRV5053, SW71 DRV5053, SW72 DRV5053, SW73 DRV5053, SW74 DRV5053, SW75 DRV5053, SW76 DRV5053, SW77 DRV5053, SW78 DRV5053, SW79 DRV5053, SW80 DRV5053, SW81 DRV5053, SW82 DRV5053

Commit message: Added photos of layout and schematic, updated Kicad files.
Connections:
- net SW74: now reaches SW74.2 (OUT)
- net SW66: now reaches SW66.2 (OUT)
- net SW59: now reaches SW59.2 (OUT)
- net SW56: now reaches SW56.2 (OUT)
- net SW46: now reaches SW46.2 (OUT)
- net SW75: now reaches SW75.2 (OUT)
- net SW57: now reaches SW57.2 (OUT)
- net SW49: now reaches SW49.2 (OUT)
- net SW82: now reaches SW82.2 (OUT)
- net SW47: now reaches SW47.2 (OUT)
- net SW43: now reaches SW43.2 (OUT)
- net SW68: now reaches SW68.2 (OUT)
- net SW76: now reaches SW76.2 (OUT)
- net SW70: now reaches SW70.2 (OUT)
- net SW63: now reaches SW63.2 (OUT)
- net SW54: now reaches SW54.2 (OUT)
- net SW72: now reaches SW72.2 (OUT)
- net SW77: now reaches SW77.2 (OUT)
- net SW69: now reaches SW69.2 (OUT)
- net SW55: now reaches SW55.2 (OUT)
- net SW42: now reaches SW42.2 (OUT)
- net SW73: now reaches SW73.2 (OUT)
- net SW80: now reaches SW80.2 (OUT)
- net SW53: now reaches SW53.2 (OUT)
- net SW50: now reaches SW50.2 (OUT)
- net SW60: now reaches SW60.2 (OUT)
- net SW64: now reaches SW64.2 (OUT)
- net SW58: now reaches SW58.2 (OUT)
- net SW62: now reaches SW62.2 (OUT)
- net SW45: now reaches SW45.2 (OUT)
- net SW65: now reaches SW65.2 (OUT)
- net SW44: now reaches SW44.2 (OUT)
- net SW61: now reaches SW61.2 (OUT)
- net SW51: now reaches SW51.2 (OUT)
- net SW79: now reaches SW79.2 (OUT)
- net SW71: now reaches SW71.2 (OUT)
- net SW81: now reaches SW81.2 (OUT)
- net SW52: now reaches SW52.2 (OUT)
- net SW67: now reaches SW67.2 (OUT)
- net SW78: now reaches SW78.2 (OUT)
- net SW48: now reaches SW48.2 (OUT)
